File: untitled.sch (EAGLE design)
At the start: 44 parts, among them IC1 LM358SO-8, IC2 LM358SO-8, Q1 STM32F439_176, T1 MOSFET-NTO220DL, T2 MOSFET-NTO220DL, T3 MOSFET-NTO220DL, T4 MOSFET-NTO220DL, T5 TRAN_NPN, T6 TRAN_NPN

Commit message: schema edited
Parts:
- added C11: 100p, ogr_lib:C0603
- added C12: 330p, ogr_lib:C0603
- added IC3: LM358SO-8, ogr_lib:LM358SO-8
- added R24: 1800, ogr_lib:R0603
- added R25: 200, ogr_lib:R0603
- added R26: 100, ogr_lib:R0603
- added R27: 22k, ogr_lib:R0603
- added T7: MOSFET-NTO220DL, ogr_lib:MOSFET-NTO220DL
- R11: value 10 -> 100
Connections:
- net N$9 renamed OZ1_OUT
- removed net N$1: C1.1, IC2A.+IN, R1.2
- removed net N$2: IC2A.OUT, R4.1
- removed net N$4: C2.2, R4.2, R5.1, T1.G
- removed net N$5: C2.1, R11.1, R15.1, R2.2, R5.2, T1.S, T3.D
- removed net ZáTěž: C4.1, R10.2, R11.2, R14.1, R7.2, T2.S, T4.D
- new net N$19: IC2A.OUT, IC3A.OUT, R26.1, R4.1
- new net N$20: C12.2, C2.2, R26.2, R27.1, R4.2, R5.1, T1.G, T7.G
- new net N$21: IC2A.-IN, IC3A.-IN, R2.1, R24.1, R25.2, R3.2
- new net ZATEZ_PIN1: C4.1, R10.2, R15.1, R7.2, T2.S, T3.D
- new net ZATEZ_PIN2: C12.1, C2.1, R14.1, R2.2, R24.2, R27.2, R5.2, T1.S, T4.D, T7.S
- net DAC2: now also R11.1
- net GND: now also C11.2, R25.1
- net N$6: now also C1.1, C11.1, IC2A.+IN, IC3A.+IN, R1.2, R11.2; no longer IC2A.-IN, R2.1, R3.2
- net VCC: now also T7.D
Other:
- note added: "Měření ADC1"
- note added: "Měření ADC2"
- note added: "Napájení OZ"
- note added: "Operační zasilovač 1 + Mosfet 1"
- note added: "Operační zasilovač 2 + Mosfet 2"
- note added: "Uzemňovací Mosfet 1"
- note added: "Uzemňovací Mosfet 2"
- moved on the sheet: C1, C10, C2, C3, C4, C5, C6, C7, C8, C9, D1, D2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

Commit message: eagle schema edited
Parts:
- removed C1, C11, C8: 100p, ogr_lib:C0603
- removed C12, C2: 330p, ogr_lib:C0603
- removed C6: 1n, ogr_lib:C0603
- removed D1: (no value), ogr_lib:D_ZENERSMA
- removed IC3: LM358SO-8, ogr_lib:LM358SO-8
- removed R1, R11, R26, R4: 100, ogr_lib:R0603
- removed R17: 56k, ogr_lib:R0603
- removed R2, R24: 1800, ogr_lib:R0603
- removed R20: 10k, ogr_lib:R0603
- removed R21: 1k, ogr_lib:R0603
- removed R22, R27, R5: 22k, ogr_lib:R0603
- removed R25, R3: 200, ogr_lib:R0603
- removed T1, T4, T7: MOSFET-NTO220DL, ogr_lib:MOSFET-NTO220DL
- removed T5: TRAN_NPN, ogr_lib:TRAN_NPN
- added C13, C16: 100p, ogr_lib:C0603
- added C14: 330p, ogr_lib:C0603
- added C15: 1n, ogr_lib:C0603
- added D3: (no value), ogr_lib:D_ZENERSMA
- added IC4: LM358SO-8, ogr_lib:LM358SO-8
- added R28, R31: 100, ogr_lib:R0603
- added R29: 1800, ogr_lib:R0603
- added R30: 200, ogr_lib:R0603
- added R32, R36: 22k, ogr_lib:R0603
- added R33: 56k, ogr_lib:R0603
- added R34: 10k, ogr_lib:R0603
- added R35: 1k, ogr_lib:R0603
- added T10: TRAN_NPN, ogr_lib:TRAN_NPN
- added T8, T9: MOSFET-N, ogr_lib:MOSFET-NTO220DL
- T2, T3: value MOSFET-NTO220DL -> MOSFET-N
Connections:
- removed net N$15: R20.2, R21.2, T5.B
- removed net N$17: C6.1, D1.K, R17.2, R22.2, T4.G, T5.C
- removed net N$19: IC2A.OUT, IC3A.OUT, R26.1, R4.1
- removed net N$20: C12.2, C2.2, R26.2, R27.1, R4.2, R5.1, T1.G, T7.G
- removed net N$21: IC2A.-IN, IC3A.-IN, R2.1, R24.1, R25.2, R3.2
- removed net N$6: C1.1, C11.1, IC2A.+IN, IC3A.+IN, R1.2, R11.2
- removed net OZ1_OUT: C4.2, R10.1, R9.2, T2.G
- new net N$10: C13.1, IC4A.+IN, R28.2
- new net N$11: IC4A.OUT, R31.1
- new net N$22: C15.1, D3.K, R33.2, R36.2, T10.C, T9.G
- new net N$23: R34.2, R35.2, T10.B
- new net N$24: C14.1, R31.2, R32.2, T8.G
- new net N$25: IC4A.-IN, R29.1, R30.2
- new net N$9: C4.1, R10.2, R9.2, T2.G
- net DAC2: now also R28.1; no longer R1.1, R11.1
- net GND: now also C13.2, C15.2, C16.2, D3.A, R30.1, R33.1, R34.1, T10.E, T9.S; no longer C1.2, C11.2, C6.2, C8.2, D1.A, R17.1, R20.1, R25.1, R3.1, T4.S, T5.E
- net GPIO2: now also C16.1, R35.1; no longer C8.1, R21.1
- net VCC: now also R36.1, T8.D; no longer R22.1, T1.D, T7.D
- net ZATEZ_PIN1: now also C4.2, R10.1; no longer C4.1, R10.2
- net ZATEZ_PIN2: now also C14.2, R29.2, R32.1, T8.S, T9.D; no longer C12.1, C2.1, R2.2, R24.2, R27.2, R5.2, T1.S, T4.D, T7.S
Other:
- note removed: "Operační zasilovač 1 + Mosfet 1"
- note removed: "Operační zasilovač 2 + Mosfet 2"
- note removed: "Uzemňovací Mosfet 1"
- note removed: "Uzemňovací Mosfet 2"
- moved on the sheet: C10, C3, C4, C5, C7, C9, D2, IC1A, IC1P, IC2P, R10, R12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
